File: sdt_qse_1496/SallenKeyFilters.kicad_sch (KiCad schematic)
At the start: 24 parts, among them U21 LM4562

Commit message: Almost ready to release Prototype 3.
Parts:
- C26: value 22uF 16V -> 22uF
- L2: value Ferrite 600 -> FerrBead
- U21: footprint Package_SO:SOIC-8-1EP_3.9x4.9mm_P1.27mm_EP2.41x3.3mm -> Package_SO:SOIC-8_3.9x4.9mm_P1.27mm
Connections:
- net TX_RAW_I_IN: now also C26.2; no longer C26.1
- net TX_RAW_Q_IN: now also C26.2; no longer C26.1
- net at R48.2, R63.2, R64.1: now also C26.1; no longer C26.2
- net at R59.2, R65.2, R66.1: now also C26.1; no longer C26.2
Other:
- note added: "This circuit provided courtesy of Rod Gatehouse AD5GH"
- title: (none) -> Sallen Key Low Pass Filters
- moved on the sheet: C26
Changed lines of the file:
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@@
 (kicad_sch (version 20230121) (generator eeschema)
   (paper "A4")
+  (title_block
+    (title "Sallen Key Low Pass Filters")
+    (date "2023-03-16")
+  )
   (junction (at 99.06 53.34) (diameter 0) (color 0 0 0 0)
   )
@@
   (wire (pts (xy 146.05 104.775) (xy 155.575 104.775))
     (stroke (width 0) (type default))
+  )
+  (text "This circuit provided courtesy of Rod Gatehouse AD5GH"
+    (at 133.35 140.335 0)
+    (effects (font (size 3 3)) (justify left bottom))
   )
   (text "Unless otherwise noted all resistors and capacitors are 1206 SMD packages.\nC21, C24, C25, C28, & C29 are 22uF 16V Tantalum, A package, Mouser 647-F931C226MAA.\nU7 is LM4562 Audio Op Amp, Mouser 926-LM4562MAX/NOPB."
@@
   (text "Transmit I&Q Audio 2nd Order Sallen-Key Low Pass Filters.  Cutoff Frequency = 11-KHz"
     (at 31.75 22.225 0)
-    (effects (font (size 1.905 1.905)) (justify left bottom))
+    (effects (font (size 3 3) (thickness 0.6) bold) (justify left bottom))
   )
   (label "12V_AA" (at 90.805 135.89 0) (fields_autoplaced)
@@
       (effects (font (size 1.27 1.27)))
     )
-    (property "Footprint" "Package_SO:SOIC-8-1EP_3.9x4.9mm_P1.27mm_EP2.41x3.3mm" (at 163.195 50.8 0)
+    (property "Footprint" "Package_SO:SOIC-8_3.9x4.9mm_P1.27mm" (at 163.195 50.8 0)
       (effects (font (size 1.27 1.27)) hide)
     )
@@
       (effects (font (size 1.27 1.27)))
     )
-    (property "Footprint" "Package_SO:SOIC-8-1EP_3.9x4.9mm_P1.27mm_EP2.41x3.3mm" (at 163.195 102.235 0)
+    (property "Footprint" "Package_SO:SOIC-8_3.9x4.9mm_P1.27mm" (at 163.195 102.235 0)
       (effects (font (size 1.27 1.27)) hide)
     )
@@
       (effects (font (size 1.27 1.27)) (justify left))
     )
-    (property "Footprint" "Package_SO:SOIC-8-1EP_3.9x4.9mm_P1.27mm_EP2.41x3.3mm" (at 74.295 144.78 0)
+    (property "Footprint" "Package_SO:SOIC-8_3.9x4.9mm_P1.27mm" (at 74.295 144.78 0)
       (effects (font (size 1.27 1.27)) hide)
     )
@@
       (effects (font (size 1.27 1.27)) (justify left))
     )
-    (property "Value" "Ferrite 600" (at 73.1012 130.683 0)
+    (property "Value" "FerrBead" (at 73.1012 130.683 0)
       (effects (font (size 1.27 1.27)) (justify left))
     )
@@
       (effects (font (size 1.27 1.27)) (justify left))
     )
-    (property "Value" "22uF 16V" (at 35.56 146.05 0)
+    (property "Value" "22uF" (at 35.56 146.05 0)
       (effects (font (size 1.27 1.27)) (justify left))
     )
@@
   (symbol (lib_id "Device:C_Polarized_Small") (at 122.555 37.465 0) (unit 1)
     (in_bom yes) (on_board yes) (dnp no) (fields_autoplaced)
-    (property "Reference" "C26" (at 125.095 36.2839 0)
-      (effects (font (size 1.27 1.27)) (justify left))
-    )
-    (property "Value" "22uF 16V" (at 125.095 38.8239 0)
+    (property "Reference" "C26" (at 125.73 36.2839 0)
+      (effects (font (size 1.27 1.27)) (justify left))
+    )
+    (property "Value" "22uF" (at 125.73 38.8239 0)
       (effects (font (size 1.27 1.27)) (justify left))
     )
@@
   (symbol (lib_id "Device:C_Polarized_Small") (at 122.555 88.9 0) (unit 1)
     (in_bom yes) (on_board yes) (dnp no) (fields_autoplaced)
-    (property "Reference" "C26" (at 125.095 87.7189 0)
-      (effects (font (size 1.27 1.27)) (justify left))
-    )
-    (property "Value" "22uF 16V" (at 125.095 90.2589 0)
+    (property "Reference" "C26" (at 125.73 87.7189 0)
+      (effects (font (size 1.27 1.27)) (justify left))
+    )
+    (property "Value" "22uF" (at 125.73 90.2589 0)
       (effects (font (size 1.27 1.27)) (justify left))
     )
@@
     )
   )
-  (symbol (lib_id "Device:C_Polarized_Small") (at 91.44 53.34 90) (unit 1)
+  (symbol (lib_id "Device:C_Polarized_Small") (at 91.44 53.34 270) (unit 1)
     (in_bom yes) (on_board yes) (dnp no) (fields_autoplaced)
-    (property "Reference" "C26" (at 90.8939 48.26 90)
-      (effects (font (size 1.27 1.27)))
-    )
-    (property "Value" "22uF 16V" (at 90.8939 50.8 90)
+    (property "Reference" "C26" (at 91.9861 48.26 90)
+      (effects (font (size 1.27 1.27)))
+    )
+    (property "Value" "22uF" (at 91.9861 50.8 90)
       (effects (font (size 1.27 1.27)))
     )
@@
     )
   )
-  (symbol (lib_id "Device:C_Polarized_Small") (at 91.44 104.775 90) (unit 1)
+  (symbol (lib_id "Device:C_Polarized_Small") (at 91.44 104.775 270) (unit 1)
     (in_bom yes) (on_board yes) (dnp no) (fields_autoplaced)
-    (property "Reference" "C26" (at 90.8939 99.695 90)
-      (effects (font (size 1.27 1.27)))
-    )
-    (property "Value" "22uF 16V" (at 90.8939 102.235 90)
-      (effects (font (size 1.27 1.27)))
-    )
+    (property "Reference" "C26" (at 91.9861 99.06 90)
+      (effects (font (size 1.27 1.27)))
+    )
+    (property "Value" "22uF" (at 91.9861 101.6 90)
+      (effects (font (size 1.27 1.27)))
+    )

Commit message: Checked gerbers, releasing to PCBWay.
Parts:
- C26: footprint Capacitor_SMD:C_1206_3216Metric -> Capacitor_Tantalum_SMD:CP_EIA-3216-10_Kemet-I
Changed lines of the file:
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@@
       (effects (font (size 1.27 1.27)) (justify left))
     )
-    (property "Footprint" "Capacitor_SMD:C_1206_3216Metric" (at 46.355 143.51 0)
+    (property "Footprint" "Capacitor_Tantalum_SMD:CP_EIA-3216-10_Kemet-I" (at 46.355 143.51 0)
       (effects (font (size 1.27 1.27)) hide)
     )
@@
       (effects (font (size 1.27 1.27)) (justify left))
     )
-    (property "Footprint" "Capacitor_SMD:C_1206_3216Metric" (at 122.555 37.465 0)
+    (property "Footprint" "Capacitor_Tantalum_SMD:CP_EIA-3216-10_Kemet-I" (at 122.555 37.465 0)
       (effects (font (size 1.27 1.27)) hide)
     )
@@
       (effects (font (size 1.27 1.27)) (justify left))
     )
-    (property "Footprint" "Capacitor_SMD:C_1206_3216Metric" (at 122.555 88.9 0)
+    (property "Footprint" "Capacitor_Tantalum_SMD:CP_EIA-3216-10_Kemet-I" (at 122.555 88.9 0)
       (effects (font (size 1.27 1.27)) hide)
     )
@@
       (effects (font (size 1.27 1.27)))
     )
-    (property "Footprint" "Capacitor_SMD:C_1206_3216Metric" (at 91.44 53.34 0)
+    (property "Footprint" "Capacitor_Tantalum_SMD:CP_EIA-3216-10_Kemet-I" (at 91.44 53.34 0)
       (effects (font (size 1.27 1.27)) hide)
     )
@@
       (effects (font (size 1.27 1.27)))
     )
-    (property "Footprint" "Capacitor_SMD:C_1206_3216Metric" (at 91.44 104.775 0)
+    (property "Footprint" "Capacitor_Tantalum_SMD:CP_EIA-3216-10_Kemet-I" (at 91.44 104.775 0)
       (effects (font (size 1.27 1.27)) hide)
     )
