File: sdt_qse_1496/sdt_qse_1496.kicad_pcb (KiCad board)
At the start: 2 copper layers, 100 x 70 mm, 117 parts, among them J1 Conn_02x08_Odd_Even, J2 SJ-3524-SMT, J3 5-1814832-1, J4 5-1814832-1, J6 Conn_01x02_Male, Q1 Q_NPN_BEC, Q2 Q_NPN_BEC, Q3 Q_PMOS_GSD, Q4 Q_PMOS_GSD, Q5 Q_NPN_BEC, Q6 Q_NPN_BEC, U1 SN74AC74PW, U2 MC1496DR2G, U3 0553-0013-BC-F, U4 LM4562, U5 MC1496DR2G

Commit message: Almost ready to release Prototype 3.
Parts:
- removed C1: 0.1uF, Capacitor_SMD:C_1206_3216Metric
- added C2: 0.1uF, Capacitor_SMD:C_1206_3216Metric, F.Cu at (179.8, 116.7)
- added J5: Conn_01x02_Male, digikey-footprints:PinHeader_1x2_P2.5mm_Drill1.1mm, F.Cu at (107.1, 93.0)
- added R1: 10k, Resistor_SMD:R_1206_3216Metric, F.Cu at (112.3, 92.8)
- added R2: 0, Resistor_SMD:R_1206_3216Metric, F.Cu at (176.6, 75.1)
- C18, C3, C32, C37, C38, C39, C40, C41, C8: value 22uF 16V -> 22uF
- C22, C5: value 25uF 25V -> 22uF
- FB1: value FerriteBead -> FerrBead
- L1: value Ferrite 600 -> FerrBead
- Q1, Q2: value Q_NPN_BEC -> NPN
- Q3, Q4: value Q_PMOS_GSD -> PMOS
- Q5, Q6: value Q_NPN_BEC -> NPN_HF
- R10, R42: value 1.3k -> 1.0k
- R11, R44: value 500 -> 470
- R26, R30: value 200 -> 220
- R31, R7: value 820 -> 1.0k
- U3: value 0553-0013-BC-F -> XFMR; footprint 0553-0013_BEL:0553-0013-BC-F -> Toroid_XFMR_SMD:Toroid_XFMR_SMD
- U4: footprint Package_SO:SOIC-8-1EP_3.9x4.9mm_P1.27mm_EP2.41x3.3mm -> Package_SO:SOIC-8_3.9x4.9mm_P1.27mm
- moved C38 62.9 mm to (142.9, 83.2), turned to -90 degrees
- moved C25 62.3 mm to (122.5, 92.5), turned to 180 degrees
- moved FB1 61.8 mm to (130.7, 113.5)
- moved C36 61.8 mm to (138.5, 84.8), turned to -90 degrees
- moved R51 58.8 mm to (146.6, 80.0), turned to -90 degrees
- moved C41 58.2 mm to (141.1, 72.3)
- moved C37 57.9 mm to (133.3, 89.8), turned to 180 degrees
- moved C33 54.5 mm to (128.7, 77.4), turned to 180 degrees
- moved R47 52.8 mm to (134.8, 84.8), turned to -90 degrees
- moved C35 52.5 mm to (125.7, 84.9), turned to 180 degrees
- moved R32 50.3 mm to (115.7, 86.8), turned to 90 degrees
- moved U4 49.9 mm to (136.0, 78.5)
- moved R54 49.0 mm to (142.9, 77.6), turned to -90 degrees
- moved R35 48.5 mm to (121.0, 87.0), turned to 90 degrees
- moved L1 47.4 mm to (128.1, 93.5), turned to 90 degrees
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Connections:
- C39 pad 1: /SallenKeyFilters/TX_RAW_I_IN -> Net-(C39-Pad1)
- C39 pad 2: Net-(C39-Pad2) -> /SallenKeyFilters/TX_RAW_I_IN
- C40 pad 1: /SallenKeyFilters/TX_RAW_Q_IN -> Net-(C40-Pad1)
- C40 pad 2: Net-(C40-Pad2) -> /SallenKeyFilters/TX_RAW_Q_IN
- R32 pad 2: Net-(C39-Pad2) -> Net-(C39-Pad1)
- R34 pad 1: Net-(C39-Pad2) -> Net-(C39-Pad1)
- R35 pad 2: Net-(C40-Pad2) -> Net-(C40-Pad1)
- R41 pad 1: Net-(C40-Pad2) -> Net-(C40-Pad1)
- R43 pad 2: Net-(C39-Pad2) -> Net-(C39-Pad1)
- R45 pad 2: Net-(C40-Pad2) -> Net-(C40-Pad1)
- U3 pad 2: /12Vswitched -> GND
- U3 pad 3: Net-(Q6-C) -> /12Vswitched
- U3 pad 4: Net-(R65-Pad2) -> unconnected-(U3-Pad4)
- U3 pad 5: unconnected-(U3-Pad5) -> Net-(Q6-C)
- U3 pad 6: GND -> Net-(R65-Pad2)
Routing:
- net Net-(Q4-D): track 97.1 -> 11.7 mm
- net /SallenKeyFilters/12V_AA: track 0.00 -> 43.6 mm, vias 0 -> 2
- net /3_3V: track 22.1 -> 49.2 mm
- net Net-(C40-Pad1): track 0.00 -> 20.9 mm, vias 0 -> 2
- net /Double Balanced Modulator1/baseband_in: track 11.8 -> 31.3 mm, vias 0 -> 2
- net Net-(C18-Pad1): track 56.2 -> 39.2 mm
- net Net-(U4B-+): track 0.00 -> 16.9 mm, vias 0 -> 2
- net /Double Balanced Modulator/baseband_in: track 11.9 -> 26.6 mm, vias 0 -> 2
- net Net-(C3-Pad1): track 37.3 -> 22.7 mm
- net Net-(U4A--): track 0.00 -> 13.7 mm
- net /12Vswitched: track 141.2 -> 152.8 mm, vias 4 -> 5
- net Net-(C39-Pad1): track 0.00 -> 11.3 mm
- net Net-(U4A-+): track 0.00 -> 11.0 mm
- net /3_3V_switched: track 83.8 -> 93.7 mm, vias 0 -> 2
- net Net-(C34-Pad2): track 0.00 -> 8.40 mm
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Other:
- board text added: "PROTOTYPE 3"
- board text removed: "PROTOTYPE 2"

Commit message: Checked gerbers, releasing to PCBWay.
Parts:
- C18, C22, C3, C32, C37, C38, C39, C40, C41, C5, C8: footprint Capacitor_SMD:C_1206_3216Metric -> Capacitor_Tantalum_SMD:CP_EIA-3216-10_Kemet-I
- C26, C27, C28, C29: value 22uF 16V -> 22uF; footprint Capacitor_SMD:C_1206_3216Metric -> Capacitor_Tantalum_SMD:CP_EIA-3216-10_Kemet-I
- R17, R18: value 5100 -> 4700
- R23, R27, R3, R5: value 1000 -> 1.0k
Routing:
- net /12Vswitched: track 152.8 -> 151.7 mm
- net /3_3V_switched: track 93.7 -> 92.6 mm
