File: sdt_qse_1496/sdt_qse_1496.kicad_sch (KiCad schematic)
At the start: 59 parts, among them J1 Conn_02x08_Odd_Even, J2 SJ-3524-SMT, J3 5-1814832-1, J4 5-1814832-1, J6 Conn_01x02_Male, Q1 Q_NPN_BEC, Q2 Q_NPN_BEC, Q3 Q_PMOS_GSD, Q4 Q_PMOS_GSD, Q5 Q_NPN_BEC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

Commit message: Almost ready to release Prototype 3.
Parts:
- removed C1: 0.1uF, Capacitor_SMD:C_1206_3216Metric, symbol Device:C_Small
- added C2: 0.1uF, Capacitor_SMD:C_1206_3216Metric, symbol Device:C_Small
- added J5: Conn_01x02_Male, digikey-footprints:PinHeader_1x2_P2.5mm_Drill1.1mm, symbol Connector:Conn_01x02_Male
- added R1: 10k, Resistor_SMD:R_1206_3216Metric, symbol Device:R_US
- added R2: 0, Resistor_SMD:R_1206_3216Metric, symbol Device:R_US
- FB1: value FerriteBead -> FerrBead
- Q1, Q2: value Q_NPN_BEC -> NPN
- Q3, Q4: value Q_PMOS_GSD -> PMOS
- Q5, Q6: value Q_NPN_BEC -> NPN_HF
- R26, R30: value 200 -> 220
- U3: value 0553-0013-BC-F -> XFMR; footprint 0553-0013_BEL:0553-0013-BC-F -> Toroid_XFMR_SMD:Toroid_XFMR_SMD
Connections:
- net 12Vswitched: now also U3.3, C2.1; no longer U3.2
- net 3_3V: now also J5.1 (Pin_1)
- net GND: now also U3.2, C2.2; no longer U3.6
- net at C17.2, Q6.3 (C): now also U3.5; no longer U3.3
- net at J3.2: now also R2.1
- net at U1.11 (2CLK), U1.3 (1CLK): now also R2.2
- net at R65.2, R66.1: now also U3.6; no longer U3.4
- net at Q1.1 (B), R49.2: now also R1.1
- new net: J5.2 (Pin_2), R1.2
Other:
- note added: "TX ON JUMPER"

Commit message: Checked gerbers, releasing to PCBWay.
Parts:
- C26, C27, C28, C29: value 22uF 16V -> 22uF; footprint Capacitor_SMD:C_1206_3216Metric -> Capacitor_Tantalum_SMD:CP_EIA-3216-10_Kemet-I
- R17, R18: value 5100 -> 4700
Changed lines of the file:
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@@
       (effects (font (size 1.27 1.27)) (justify left))
     )
-    (property "Value" "22uF 16V" (at 256.54 105.4989 0)
+    (property "Value" "22uF" (at 256.54 105.4989 0)
       (effects (font (size 1.27 1.27)) (justify left))
     )
-    (property "Footprint" "Capacitor_SMD:C_1206_3216Metric" (at 254 104.14 0)
+    (property "Footprint" "Capacitor_Tantalum_SMD:CP_EIA-3216-10_Kemet-I" (at 254 104.14 0)
       (effects (font (size 1.27 1.27)) hide)
     )
@@
   (symbol (lib_id "Device:C_Polarized_Small") (at 226.06 154.94 0) (unit 1)
     (in_bom yes) (on_board yes) (dnp no) (fields_autoplaced)
-    (property "Reference" "C27" (at 228.219 153.5592 0)
+    (property "Reference" "C27" (at 228.6 153.7589 0)
       (effects (font (size 1.27 1.27)) (justify left))
     )
-    (property "Value" "22uF 16V" (at 228.219 156.0961 0)
+    (property "Value" "22uF" (at 228.6 156.2989 0)
       (effects (font (size 1.27 1.27)) (justify left))
     )
-    (property "Footprint" "Capacitor_SMD:C_1206_3216Metric" (at 226.06 154.94 0)
+    (property "Footprint" "Capacitor_Tantalum_SMD:CP_EIA-3216-10_Kemet-I" (at 226.06 154.94 0)
       (effects (font (size 1.27 1.27)) hide)
     )
@@
       (effects (font (size 1.27 1.27)) (justify left))
     )
-    (property "Value" "22uF 16V" (at 256.54 119.4689 0)
+    (property "Value" "22uF" (at 256.54 119.4689 0)
       (effects (font (size 1.27 1.27)) (justify left))
     )
-    (property "Footprint" "Capacitor_SMD:C_1206_3216Metric" (at 254 118.11 0)
+    (property "Footprint" "Capacitor_Tantalum_SMD:CP_EIA-3216-10_Kemet-I" (at 254 118.11 0)
       (effects (font (size 1.27 1.27)) hide)
     )
@@
     )
     (pin "1")
+    (pin "2")
     (pin "3")
+    (pin "4")
     (pin "5")
     (pin "6")
-    (pin "4")
-    (pin "2")
     (instances
       (project "sdt_qse_1496"
@@
       (effects (font (size 1.27 1.27)) (justify left))
     )
-    (property "Value" "22uF 16V" (at 227.33 133.4389 0)
+    (property "Value" "22uF" (at 227.33 133.4389 0)
       (effects (font (size 1.27 1.27)) (justify left))
     )
-    (property "Footprint" "Capacitor_SMD:C_1206_3216Metric" (at 224.79 132.08 0)
+    (property "Footprint" "Capacitor_Tantalum_SMD:CP_EIA-3216-10_Kemet-I" (at 224.79 132.08 0)
       (effects (font (size 1.27 1.27)) hide)
     )
@@
   (symbol (lib_id "Device:R_US") (at 167.64 55.88 180) (unit 1)
     (in_bom yes) (on_board yes) (dnp no) (fields_autoplaced)
-    (property "Reference" "R17" (at 169.291 55.0453 0)
-      (effects (font (size 1.27 1.27)) (justify right))
-    )
-    (property "Value" "5100" (at 169.291 57.5822 0)
+    (property "Reference" "R17" (at 170.18 55.245 0)
+      (effects (font (size 1.27 1.27)) (justify right))
+    )
+    (property "Value" "4700" (at 170.18 57.785 0)
       (effects (font (size 1.27 1.27)) (justify right))
     )
@@
   (symbol (lib_id "Device:R_US") (at 167.64 104.14 180) (unit 1)
     (in_bom yes) (on_board yes) (dnp no) (fields_autoplaced)
-    (property "Reference" "R18" (at 169.291 103.3053 0)
-      (effects (font (size 1.27 1.27)) (justify right))
-    )
-    (property "Value" "5100" (at 169.291 105.8422 0)
-      (effects (font (size 1.27 1.27)) (justify right))
-    )
+    (property "Reference" "R18" (at 170.18 103.505 0)
+      (effects (font (size 1.27 1.27)) (justify right))
+    )
+    (property "Value" "4700" (at 170.18 106.045 0)
+      (effects (font (size 1.27 1.27)) (justify right))
+    )
